File: pcb/keyboard.kicad_pcb (KiCad board)
At the start: 2 copper layers, 356.5 x 123.6 mm, 132 parts, among them SW1 SW_Push_45deg, SW10 SW_Push_45deg, SW11 SW_Push_45deg, SW12 SW_Push_45deg, SW13 SW_Push_45deg, SW14 SW_Push_45deg, SW15 SW_Push_45deg, SW16 SW_Push_45deg, SW17 SW_Push_45deg, SW18 SW_Push_45deg, SW19 SW_Push_45deg, SW2 SW_Push_45deg, SW20 SW_Push_45deg, SW21 SW_Push_45deg, SW22 SW_Push_45deg, SW23 SW_Push_45deg, SW24 SW_Push_45deg, SW25 SW_Push_45deg, SW26 SW_Push_45deg, SW27 SW_Push_45deg, SW28 SW_Push_45deg, SW29 SW_Push_45deg, SW3 SW_Push_45deg, SW30 SW_Push_45deg, SW31 SW_Push_45deg, SW32 SW_Push_45deg, SW33 SW_Push_45deg, SW34 SW_Push_45deg, SW35 SW_Push_45deg, SW36 SW_Push_45deg, SW37 SW_Push_45deg, SW38 SW_Push_45deg, SW39 SW_Push_45deg, SW4 SW_Push_45deg, SW40 SW_Push_45deg, SW41 SW_Push_45deg, SW42 SW_Push_45deg, SW43 SW_Push_45deg, SW44 SW_Push_45deg, SW45 SW_Push_45deg, SW46 SW_Push_45deg, SW47 SW_Push_45deg, SW48 SW_Push_45deg, SW49 SW_Push_45deg, SW5 SW_Push_45deg, SW50 SW_Push_45deg, SW51 SW_Push_45deg, SW52 SW_Push_45deg, SW53 SW_Push_45deg, SW54 SW_Push_45deg, SW55 SW_Push_45deg, SW56 SW_Push_45deg, SW57 SW_Push_45deg, SW58 SW_Push_45deg, SW59 SW_Push_45deg, SW6 SW_Push_45deg, SW60 SW_Push_45deg, SW61 SW_Push_45deg, SW62 SW_Push_45deg, SW63 SW_Push_45deg, SW64 SW_Push_45deg, SW65 SW_Push_45deg, SW7 SW_Push_45deg, SW77 RotaryEncoder_Switch, SW8 SW_Push_45deg, SW9 SW_Push_45deg

Commit message: Add all PCB files
Parts:
- D2: moved to B.Cu
- SW1, SW10, SW11, SW12, SW13, SW16, SW17, SW18, SW19, SW2, SW20, SW21, SW22, SW23, SW24, SW25, SW26, SW27, SW3, SW30, SW31, SW32, SW33, SW34, SW35, SW36, SW37, SW38, SW39, SW4, SW40, SW43, SW44, SW45, SW46, SW47, SW48, SW49, SW5, SW50, SW51, SW52, SW6, SW62, SW63, SW64, SW65, SW7, SW8, SW9: footprint Hotswap Sockets:MX-Hotswap-1U -> PCM_Switch_Keyboard_Hotswap_Kailh:SW_Hotswap_Kailh_MX_1.00u; moved to F.Cu
- SW14: footprint Hotswap Sockets:MX-Hotswap-2U -> PCM_Switch_Keyboard_Hotswap_Kailh:SW_Hotswap_Kailh_MX_2.00u; moved to F.Cu
- SW15, SW28: footprint Hotswap Sockets:MX-Hotswap-1.5U -> PCM_Switch_Keyboard_Hotswap_Kailh:SW_Hotswap_Kailh_MX_1.50u; moved to F.Cu
- SW29: footprint Hotswap Sockets:MX-Hotswap-1.75U -> PCM_Switch_Keyboard_Hotswap_Kailh:SW_Hotswap_Kailh_MX_1.75u; moved to F.Cu
- SW41, SW42: footprint Hotswap Sockets:MX-Hotswap-2.25U -> PCM_Switch_Keyboard_Hotswap_Kailh:SW_Hotswap_Kailh_MX_2.25u; moved to F.Cu
- SW53: footprint Hotswap Sockets:MX-Hotswap-2.75U -> PCM_Switch_Keyboard_Hotswap_Kailh:SW_Hotswap_Kailh_MX_2.75u; moved to F.Cu
- SW54, SW55, SW56, SW58, SW59, SW60, SW61: footprint Hotswap Sockets:MX-Hotswap-1.25U -> PCM_Switch_Keyboard_Hotswap_Kailh:SW_Hotswap_Kailh_MX_1.25u; moved to F.Cu
- SW57: footprint Hotswap Sockets:MX-Hotswap-6.25U -> PCM_Switch_Keyboard_Hotswap_Kailh:SW_Hotswap_Kailh_MX_6.25u; moved to F.Cu
- moved D12 1.04 mm to (265.8, 78.5)
- moved D2 0.23 mm to (74.9, 78.5)
- turned SW1 to 0 degrees
- turned SW10 to 0 degrees
- turned SW11 to 0 degrees
- turned SW12 to 0 degrees
- turned SW13 to 0 degrees
- turned SW14 to 0 degrees
- turned SW15 to 0 degrees
- turned SW16 to 0 degrees
- turned SW17 to 0 degrees
- turned SW18 to 0 degrees
- turned SW19 to 0 degrees
- turned SW2 to 0 degrees
- turned SW20 to 0 degrees
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Routing:
- net Net-(A1-GPIO22): track 387.8 -> 317.0 mm
- net ROW2: track 410.8 -> 373.1 mm
- net ROW4: track 461.0 -> 427.8 mm
- net ROW1: track 420.9 -> 388.3 mm
- net COL1: track 413.0 -> 441.7 mm
- net COL14: track 144.8 -> 170.8 mm
- net GND: track 403.6 -> 423.0 mm
- net COL2: track 401.0 -> 420.1 mm
- net ROW3: track 409.9 -> 399.2 mm
- net Net-(A1-GPIO14): track 350.6 -> 340.8 mm
- net COL3: track 391.3 -> 400.4 mm
- net COL8: track 268.1 -> 277.1 mm
- net COL7: track 288.0 -> 296.6 mm
- net COL15: track 103.2 -> 94.9 mm
- net COL5: track 325.7 -> 333.7 mm
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Other:
- board text added: "AGND Plane"
- board text added: "Copper"
- board text added: "Exposed"
- board text added: "Exposed Copper Keep Out"
- board text added: "Keep"
- board text added: "Keep Out"
- board text added: "Out"
- board text added: "USB Cable"
- board text added: "arjun's keyboard"

Commit message: updated pcb files
Connections:
- A1 pad 27: ROW6 -> COL15
- A1 pad 35: COL15 -> unconnected-(A1-ADC_VREF-Pad35)
Routing:
- net COL15: track 94.9 -> 75.6 mm
Changed lines of the file:
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@@
 		(pcbplotparams
 			(layerselection 0x00000000_00000000_55555555_5755f5ff)
-			(plot_on_all_layers_selection 0x00000000_00000000_00000000_00000000)
+			(plot_on_all_layers_selection 0x00000000_00000000_00000000_0200a0af)
 			(disableapertmacros no)
 			(usegerberextensions no)
@@
 			(outputformat 1)
 			(mirror no)
-			(drillshape 1)
+			(drillshape 0)
 			(scaleselection 1)
-			(outputdirectory "")
+			(outputdirectory "keyboard-gerber")
 		)
 	)
@@
 	(net 23 "ROW3")
 	(net 24 "unconnected-(A1-3V3_EN-Pad37)")
-	(net 25 "ROW6")
+	(net 25 "unconnected-(A1-ADC_VREF-Pad35)")
 	(net 26 "ROW4")
 	(net 27 "unconnected-(A1-3V3-Pad36)")
@@
 			(layers "*.Cu" "*.Mask")
 			(remove_unused_layers no)
-			(net 25 "ROW6")
+			(net 5 "COL15")
 			(pinfunction "GPIO21")
 			(pintype "bidirectional")
@@
 			(layers "F.Cu" "F.Mask")
 			(roundrect_rratio 0.5)
-			(net 25 "ROW6")
+			(net 5 "COL15")
 			(pinfunction "GPIO21")
 			(pintype "bidirectional")
@@
 			(layers "*.Cu" "*.Mask")
 			(remove_unused_layers no)
-			(net 5 "COL15")
+			(net 25 "unconnected-(A1-ADC_VREF-Pad35)")
 			(pinfunction "ADC_VREF")
 			(pintype "power_in")
@@
 			(layers "F.Cu" "F.Mask")
 			(roundrect_rratio 0.5)
-			(net 5 "COL15")
+			(net 25 "unconnected-(A1-ADC_VREF-Pad35)")
 			(pinfunction "ADC_VREF")
 			(pintype "power_in")
@@
 	)
 	(segment
-		(start 381.05875 52.27)
-		(end 377.89 49.10125)
+		(start 381.05875 70.865)
+		(end 379.615 69.42125)
 		(width 0.2)
 		(layer "B.Cu")
@@
 	(segment
 		(start 381.05875 142.71625)
-		(end 381.05875 52.27)
+		(end 381.05875 70.865)
+		(width 0.2)
+		(layer "B.Cu")
+		(net 5)
+	)
+	(segment
+		(start 379.615 69.42125)
+		(end 377.89 69.42125)
 		(width 0.2)
 		(layer "B.Cu")
