File: pcb/keyboard.kicad_sch (KiCad schematic)
At the start: 132 parts, among them SW1 SW_Push_45deg, SW10 SW_Push_45deg, SW11 SW_Push_45deg, SW12 SW_Push_45deg, SW13 SW_Push_45deg, SW14 SW_Push_45deg, SW15 SW_Push_45deg, SW16 SW_Push_45deg, SW17 SW_Push_45deg, SW18 SW_Push_45deg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

Commit message: updated pcb files
Connections:
- net ROW6 is gone; now on net COL15: A1.27 (GPIO21)
- net COL15: no longer A1.35 (ADC_VREF)
